File: PCB-v1/PCB-v1.kicad_pcb (KiCad board)
At the start: 2 copper layers, 37 x 37.5 mm, 8 parts, among them Q1 2N2222, U1 XIAO ESP32C3

Commit message: ADD BOM
Parts:
- B1: footprint Connector_PinHeader_2.54mm:PinHeader_1x02_P2.54mm_Vertical -> Connector_PinHeader_1.00mm:PinHeader_1x02_P1.00mm_Horizontal
Connections:
- M1 pad 1: Net-(M1-VIN) -> unconnected-(M1-SHUT-Pad1)
- M1 pad 2: Net-(M1-GND) -> unconnected-(M1-INT-Pad2)
- M1 pad 5: unconnected-(M1-INT-Pad5) -> Net-(M1-GND)
- M1 pad 6: unconnected-(M1-SHUT-Pad6) -> Net-(M1-VIN)
Routing:
- net Net-(M1-VIN): track 63.4 -> 81.0 mm
- net Net-(M1-GND): track 26.6 -> 35.1 mm
- net Net-(M1-SDA): track 18.8 -> 15.9 mm
- net Net-(B1--): track 5.73 -> 4.36 mm
