File: PCB-v1/PCB-v1.kicad_sch (KiCad schematic)
At the start: 8 parts, among them Q1 2N2222, U1 XIAO ESP32C3

Commit message: ADD BOM
Parts:
- B1: footprint Connector_PinHeader_2.54mm:PinHeader_1x02_P2.54mm_Vertical -> Connector_PinHeader_1.00mm:PinHeader_1x02_P1.00mm_Horizontal; Link (none) -> https://www.amazon.com/YTKavq-Battery-Lithium-Rechargeable-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; Supplier (none) -> Amazon
- LS1: Link (none) -> https://www.aliexpress.us/item/3256808371712170.html?utpara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; Supplier (none) -> Aliexpress
- M1: Link (none) -> https://www.aliexpress.us/item/3256806005285334.html?utpara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; Mounting header link (none) -> https://www.aliexpress.us/item/3256807353673955.html?utpara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; Supplier (none) -> Aliexpress
- Q1: Link (none) -> https://www.aliexpress.us/item/3256807891334673.html?utpara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; Supplier (none) -> Aliexpress
- R1, R2, R3: Link (none) -> https://www.amazon.com/Avelis-Resistors-Assortment-Precisio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; Supplier (none) -> Amazon
- U1: footprint esp:xiao_esp32c3 -> XIAO_ESP32C3:xiao_esp32c3; Link (none) -> https://www.seeedstudio.com/Seeed-Studio-XIAO-ESP32C3-Tape-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; Quantity (none) -> 1; SKU (none) -> 101991467; Supplier (none) -> Seeed Technology
Connections:
- net at Q1.1, U1.13 (GND): now also M1.5 (GND); no longer M1.2 (GND)
- net at LS1.2, U1.12 (VCC_3V3): now also M1.6 (VIN); no longer M1.1 (VIN)
